Commit message: Taske

File: my_rb1_description/urdf/my_rb1_robot.xacro (robot description, xacro)
@@ -37,5 +37,4 @@
         <child link="base_link" />
         <parent link="base_footprint" />
-        <joint_properties damping="1.0" friction="1.0" />
     </joint>
         <!-- Link - base_link -->
@@ -71,7 +70,5 @@
         <child link="left_wheel" />
         <parent link="base_link" />
-        <axis rpy="0 0 0" xyz="0 1 0" />
-        <limit effort="10000" velocity="1000" />
-        <joint_properties damping="1.0" friction="1.0" />
+        <!--<axis rpy="0 0 0" xyz="0 1 0" />-->
     </joint>
       <!-- Link - link_left_wheel -->
@@ -108,7 +105,5 @@
         <child link="right_wheel" />
         <parent link="base_link" />
-        <axis rpy="0 0 0" xyz="0 1 0" />
-        <limit effort="10000" velocity="1000" />
-        <joint_properties damping="1.0" friction="1.0" />
+        <!--<axis rpy="0 0 0" xyz="0 1 0" />-->
     </joint>
           <!-- Link - link_right_wheel -->
@@ -145,6 +140,4 @@
         <child link="front_caster" />
         <parent link="base_link" />
-        <limit effort="10000" velocity="1000" />
-        <joint_properties damping="1.0" friction="1.0" />
     </joint>
      <!-- Link - front_caster_wheel -->
@@ -180,6 +173,4 @@
         <child link="back_caster" />
         <parent link="base_link" />
-        <limit effort="10000" velocity="1000" />
-        <joint_properties damping="1.0" friction="1.0" />
     </joint>
          <!-- Link - back_caster_wheel -->
@@ -211,9 +202,8 @@
     </link>
         <!-- Laser scan -->
-    <joint name="joint_front_laser_chassis" type="fixed">
+    <joint name="joint_front_laser_base_link" type="fixed">
         <origin rpy="3.14 0 0" xyz="0.25 0.0 0.075"/>
         <child link="front_laser" />
         <parent link="base_link" />
-        <joint_properties damping="1.0" friction="1.0" />
     </joint>
     <link name="front_laser">

Commit message: Checkpoint:2_Rotate_Robot

File: my_rb1_description/urdf/my_rb1_robot.xacro (robot description, xacro)
@@ -2,230 +2,173 @@
 <robot name="robot" xmlns:xacro="http://www.ros.org/wiki/xacro">
     <xacro:include filename="$(find my_rb1_description)/urdf/my_rb1_robot.gazebo" />
-    <!-- Parameters -->
-    <!--<xacro:property name="chassis_mass" value="10" />
-    <xacro:property name="pi" value="3.1415926535897931"/>-->
-    	    <!-- Link - base_footprint -->
+    <!-- Define materials for visualization -->
+    <material name="blue">
+        <color rgba="0 0 1 1"/>
+    </material>
+    <material name="gray">
+        <color rgba="0.40 0.40 0.40 1"/>
+    </material>
+    <material name="red">
+        <color rgba="1 0 0 1"/>
+    </material>
+    <!-- Base footprint link -->
     <link name="base_footprint">
+    </link>
+    <!-- Joint connecting base_link and base_footprint -->
+    <joint name="base_link_plate_joint" type="fixed">
+        <origin rpy="0 0 0" xyz="0 0 0.15" />
+        <parent link="base_footprint" />
+        <child link="base_link" />
+    </joint>
+    <!-- Base link -->
+    <link name="base_link">
+        <!-- Visual representation of the base link -->
+        <visual>
+            <origin xyz="0 0 0" rpy="0 0 0"/>
+            <geometry>
+                <cylinder radius="0.25" length="0.3"/>
+            </geometry>
+            <material name="blue"/>
+        </visual>
+        <!-- Collision representation of the base link -->
+        <collision>
+            <origin xyz="0 0 0" rpy="0 0 0"/>
+            <geometry>
+                <cylinder radius="0.25" length="0.3"/>
+            </geometry>
+        </collision>
+        <!-- Inertial properties of the base link -->
         <inertial>
-            <mass value="1" />
-            <origin xyz="0 0 0.5" rpy="0 0 0" />
-            <inertia ixx="0.37505" ixy="0" ixz="0" iyy="0.37505" iyz="0" izz="0.125" />
+            <mass value="20.5" />
+            <origin xyz="0 0 0" rpy="0 0 0" />
+            <inertia ixx="0.47406249999999994" ixy="0.0" ixz="0.0" iyy="0.47406249999999994" iyz="0.0" izz="0.640625" />
         </inertial>
+    </link>
+    <!-- Left wheel link -->
+    <link name="left_wheel">
+        <!-- Visual representation of the left wheel -->
+        <visual>
+            <origin xyz="0 0 0" rpy="-1.575 0 0"/>
+            <geometry>
+                <cylinder radius="0.025" length="0.03"/>
+            </geometry>
+            <material name="red"/>
+        </visual>
+        <!-- Collision representation of the left wheel -->
         <collision>
+            <origin xyz="0 0 0" rpy="-1.575 0 0"/>
             <geometry>
-                <cylinder length="0.01" radius="0.25"/>
+                <cylinder radius="0.025" length="0.03"/>
             </geometry>
-            <!--<geometry>
-                <mesh filename="package://robot_description/meshes/chassis.stl" />
-            </geometry>-->
         </collision>
+        <!-- Inertial properties of the left wheel -->
+        <inertial>
+            <mass value="1.5" />
+            <origin xyz="0 0 0" rpy="-1.575 0 0" />
+            <inertia ixx="0.00034687500000000007" ixy="0.0" ixz="0.0" iyy="0.00034687500000000007" iyz="0.0" izz="0.0004687500000000001" />
+        </inertial>
+    </link>
+    <!-- Joint connecting base_link and left_wheel -->
+    <joint name="base_link_left_wheel_joint" type="continuous">
+        <axis xyz="0 1 0" rpy="0 0 0" />
+        <origin rpy="0 0 0" xyz="0 0.2 -0.15" />
+        <parent link="base_link" />
+        <child link="left_wheel" />
+    </joint>
+    <!-- Right wheel link -->
+    <link name="right_wheel">
+        <!-- Visual representation of the right wheel -->
         <visual>
+            <origin xyz="0 0 0" rpy="-1.575 0 0"/>
             <geometry>
-                <cylinder length="0.01" radius="0.25"/>
+                <cylinder radius="0.025" length="0.03"/>
             </geometry>
-            <!-- <geometry>
-                <box size="2 1.3 0.4" />
-            </geometry> -->
-            <material name="DarkBlue">
-                <color rgba="0.2 0.2 0.4 1" />
-            </material>
+            <material name="red"/>
         </visual>
+        <!-- Collision representation of the right wheel -->
+        <collision>
+            <origin xyz="0 0 0" rpy="-1.575 0 0"/>
+            <geometry>
+                <cylinder radius="0.025" length="0.03"/>
+            </geometry>
+        </collision>
+        <!-- Inertial properties of the right wheel -->
+        <inertial>
+            <mass value="1.5" />
+            <origin xyz="0 0 0" rpy="-1.575 0 0" />
+            <inertia ixx="0.00034687500000000007" ixy="0.0" ixz="0.0" iyy="0.00034687500000000007" iyz="0.0" izz="0.0004687500000000001" />
+        </inertial>
     </link>
-     <!-- Joint - base_link -->
-    <joint name="joint_footprint_base_link" type="fixed">
-        <origin rpy="0 0 0" xyz="0 0 0.15" />
-        <child link="base_link" />
-        <parent link="base_footprint" />
+    <!-- Joint connecting base_link and right_wheel -->
+    <joint name="base_link_right_wheel_joint" type="continuous">
+        <axis xyz="0 1 0" rpy="0 0 0" />
+        <origin rpy="0 0 0" xyz="0 -0.2 -0.15" />
+        <parent link="base_link" />
+        <child link="right_wheel" />
     </joint>
-        <!-- Link - base_link -->
-    <link name="base_link">
-        <inertial>
-            <mass value="19" />
-            <origin xyz="0 0 0" rpy="0 0 0" />
-            <inertia ixx="0.677" ixy="0" ixz="0" iyy="0.677" iyz="0" izz="0.59375" />
-        </inertial>
-        <collision>
-            <geometry>
-                <cylinder length="0.29" radius="0.25"/>
-            </geometry>
-            <!--<geometry>
-                <mesh filename="package://robot_description/meshes/chassis.stl" />
-            </geometry>-->
-        </collision>
-        <visual>
-             <geometry>
-                <cylinder length="0.29" radius="0.25"/>
-            </geometry>
-            <!-- <geometry>
-                <box size="2 1.3 0.4" />
-            </geometry> -->
-            <material name="DarkBlue">
-                <color rgba="0.2 0.2 0.4 1" />
-            </material>
-        </visual>
-    </link>
-         <!-- Joint - base_link / left wheel -->
-    <joint name="joint_base_link_left_wheel" type="continuous">
-        <origin rpy="0 0 0" xyz="0.0 -0.2 -0.15" />
-        <child link="left_wheel" />
-        <parent link="base_link" />
-        <!--<axis rpy="0 0 0" xyz="0 1 0" />-->
-    </joint>
-      <!-- Link - link_left_wheel -->
-    <link name="left_wheel">
-        <inertial>
-            <mass value="1" />
-            <origin xyz="0 -0.2 0.5" rpy="1.5707 0 0" />
-            <inertia ixx="0.0002083" ixy="0" ixz="0" iyy="0.0003125" iyz="0" izz="0.0002083" />
-        </inertial>
-        <collision>
-            <geometry>
-                <cylinder length="0.025" radius="0.025"/>
-            </geometry>
-            <!--<geometry>
-                <mesh filename="package://robot_description/meshes/chassis.stl" />
-            </geometry>-->
-        </collision>
-        <visual>
-         <origin xyz="0 0 0" rpy="1.5707 0 0" />
-             <geometry>
-                <cylinder length="0.025" radius="0.025"/>
-            </geometry>
-            <!-- <geometry>
-                <box size="2 1.3 0.4" />
-            </geometry> -->
-            <!--<material name="DarkBlue">
-                <color rgba="0.2 0.2 0.4 1" />
-            </material>-->
-        </visual>
-    </link>
-            <!-- Joint - base_link / right wheel -->
-    <joint name="joint_base_link_right_wheel" type="continuous">
-        <origin rpy="0 0 0" xyz="0.0 0.2 -0.15" />
-        <child link="right_wheel" />
-        <parent link="base_link" />
-        <!--<axis rpy="0 0 0" xyz="0 1 0" />-->
-    </joint>
-          <!-- Link - link_right_wheel -->
-    <link name="right_wheel">
-        <inertial>
-            <mass value="1" />
-            <origin xyz="0 0.2 0.5" rpy="1.5707 0 0" />
-            <inertia ixx="0.0002083" ixy="0" ixz="0" iyy="0.0003125" iyz="0" izz="0.0002083" />
-        </inertial>
-        <collision>
-            <geometry>
-                <cylinder length="0.025" radius="0.025"/>
-            </geometry>
-            <!--<geometry>
-                <mesh filename="package://robot_description/meshes/chassis.stl" />
-            </geometry>-->
-        </collision>
-        <visual>
-         <origin xyz="0 0 0" rpy="1.5707 0 0" />
-             <geometry>
-                <cylinder length="0.025" radius="0.025"/>
-            </geometry>
-            <!-- <geometry>
-                <box size="2 1.3 0.4" />
-            </geometry> -->
-            <!--<material name="DarkBlue">
-                <color rgba="0.2 0.2 0.4 1" />
-            </material>-->
-        </visual>
-    </link>
-             <!-- Joint - base_link / front caster wheel -->
-    <joint name="joint_base_link_front_caster_wheel" type="fixed">
-        <origin rpy="0 0 0" xyz="0.1 0.0 -0.15" />
-        <child link="front_caster" />
-        <parent link="base_link" />
-    </joint>
-     <!-- Link - front_caster_wheel -->
+    <!-- Link representing the front caster wheel -->
     <link name="front_caster">
-        <inertial>
-            <mass value="1" />
-            <origin xyz="0.1 0.0 0.5" rpy="0 0 0" />
-            <inertia ixx="0.00025" ixy="0" ixz="0" iyy="0.00025" iyz="0" izz="0.00025" />
-        </inertial>
-        <collision>
-            <geometry>
-                <sphere radius="0.025"/>
-            </geometry>
-            <!--<geometry>
-                <mesh filename="package://robot_description/meshes/chassis.stl" />
-            </geometry>-->
-        </collision>
-        <visual>
-             <geometry>
-                 <sphere radius="0.025"/>
-            </geometry>
-            <!-- <geometry>
-                <box size="2 1.3 0.4" />
-            </geometry> -->
-           <material name="dark_grey">
-            <color rgba="0.662745 0.662745 0.662745 1.0"/>
-            </material>
-        </visual>
-    </link>
-        <!-- Joint - base_link / back caster wheel -->
-        <joint name="joint_base_link_back_caster_wheel" type="fixed">
-        <origin rpy="0 0 0" xyz="-0.1 0.0 -0.15" />
-        <child link="back_caster" />
-        <parent link="base_link" />
-    </joint>
-         <!-- Link - back_caster_wheel -->
-    <link name="back_caster">
-        <inertial>
-            <mass value="1" />
-            <origin xyz="-0.1 0.0 0.5" rpy="0 0 0" />
-            <inertia ixx="0.00025" ixy="0" ixz="0" iyy="0.00025" iyz="0" izz="0.00025" />
-        </inertial>
-        <collision>
-            <geometry>
-                <sphere radius="0.025"/>
-            </geometry>
-            <!--<geometry>
-                <mesh filename="package://robot_description/meshes/chassis.stl" />
-            </geometry>-->
-        </collision>
-        <visual>
-             <geometry>
-                 <sphere radius="0.025"/>
-            </geometry>
-            <!-- <geometry>
-                <box size="2 1.3 0.4" />
-            </geometry> -->
-            <material name="dark_grey">
-                <color rgba="0.662745 0.662745 0.662745 1.0"/>
-            </material>
-        </visual>
-    </link>
-        <!-- Laser scan -->
-    <joint name="joint_front_laser_base_link" type="fixed">
-        <origin rpy="3.14 0 0" xyz="0.25 0.0 0.075"/>
-        <child link="front_laser" />
-        <parent link="base_link" />
-    </joint>
-    <link name="front_laser">
-        <inertial>
-            <origin xyz="0 0 0" rpy="0 0 0" />
-            <mass value="1" />
-            <inertia ixx="0.000133" ixy="0" ixz="0" iyy="0.000133" iyz="0" izz="0.0002"/>
-        </inertial>
         <visual>
             <origin xyz="0 0 0" rpy="0 0 0" />
             <geometry>
-                <cylinder radius="0.02" length="0.02"/>
+                <sphere radius="0.025" />
             </geometry>
-            <material name="Red">
-                <color rgba="0.7 0.1 0.1 1" />
-            </material>
+            <material name="gray"/>
         </visual>
         <collision>
-            <origin xyz="0 0 0" rpy="0 0 0"/>
+            <origin xyz="0 0 0" rpy="0 0 0" />
+            <contact_coefficients mu="0.0" kp="0.0" kd="0.0" />
             <geometry>
-                <cylinder radius="0.02" length="0.02"/>
+                <sphere radius="0.025" />
             </geometry>
         </collision>
+        <inertial>
+            <mass value="0.5" />
+            <origin xyz="0 0 0" rpy="0 0 0" />
+            <inertia ixx="0.00012500000000000003" ixy="0.0" ixz="0.0" iyy="0.00012500000000000003" iyz="0.0" izz="0.00012500000000000003" />
+        </inertial>
     </link>
+    <!-- Joint connecting base_link and front_caster -->
+    <joint name="base_link_front_caster_joint" type="fixed">
+        <parent link="base_link"/>
+        <child link="front_caster"/>
+        <origin xyz="0.1 0.0 -0.15" rpy="0 0 0"/>
+    </joint>
+    <!-- Link representing the back caster wheel -->
+    <link name="back_caster">
+        <visual>
+            <origin xyz="0 0 0" rpy="0 0 0" />
+            <geometry>
+                <sphere radius="0.025" />
+            </geometry>
+            <material name="gray"/>
+        </visual>
+        <collision>
+            <origin xyz="0 0 0" rpy="0 0 0" />
+            <contact_coefficients mu="0.0" kp="0.0" kd="0.0" />
+            <geometry>
+                <sphere radius="0.025" />
+            </geometry>
+        </collision>
+        <inertial>
+            <mass value="0.5" />
+            <origin xyz="0 0 0" rpy="0 0 0" />
+            <inertia ixx="0.00012500000000000003" ixy="0.0" ixz="0.0" iyy="0.00012500000000000003" iyz="0.0" izz="0.00012500000000000003" />
+        </inertial>
+    </link>
+    <!-- Joint connecting base_link and back_caster -->
+    <joint name="base_link_back_caster_joint" type="fixed">
+        <parent link="base_link"/>
+        <child link="back_caster"/>
+        <origin xyz="-0.1 0.0 -0.15" rpy="0 0 0"/>
+    </joint>
+    <!-- Link representing the laser -->
+    <link name="front_laser">
+    </link>
+    <!-- Joint connecting base_link and front_laser -->
+    <joint name="base_link_front_laser_joint" type="fixed">
+        <origin rpy="3.14 0 0" xyz="0.25 0 0.075" />
+        <parent link="base_link" />
+        <child link="front_laser" />
+    </joint>
 </robot>
